Commit message: Update sim launch and hexapod xacro
Co-Authored-By: Claude Sonnet 5 <noreply@anthropic.com>

File: backup_camvis/src/hexapod_description/urdf/hexapod.urdf.xacro (robot description, xacro)
@@ -29,7 +29,4 @@
   <xacro:arg name="use_camera"   default="true"/>
   <xacro:arg name="use_joint_ft" default="true"/>
-  <!-- camera_visual:=false hides the depth-camera box (visual only - collision, mass and the
-       sensor stay), e.g. for figure screenshots (scripts/capture_figures.sh). -->
-  <xacro:arg name="camera_visual" default="true"/>
   <!-- Battery + boards inside the body (masses from tools/mass_budget.yaml). false = bare CAD robot -->
   <xacro:arg name="use_electronics" default="true"/>

File: backup_camvis/src/hexapod_description/urdf/sensors.xacro (robot description, xacro)
@@ -20,11 +20,9 @@
   <xacro:property name="csz" value="${float(cs[2])}"/>
   <link name="camera_link">
-    <xacro:if value="$(arg camera_visual)">
-      <visual>
-        <origin xyz="${-csx/2} 0 0" rpy="0 0 0"/>
-        <geometry><box size="${csx} ${csy} ${csz}"/></geometry>
-        <material name="sensor_blue"/>
-      </visual>
-    </xacro:if>
+    <visual>
+      <origin xyz="${-csx/2} 0 0" rpy="0 0 0"/>
+      <geometry><box size="${csx} ${csy} ${csz}"/></geometry>
+      <material name="sensor_blue"/>
+    </visual>
     <collision>
       <origin xyz="${-csx/2} 0 0" rpy="0 0 0"/>
